File: sideA.sch (KiCad schematic (older format))
At the start: 0 parts

Commit message: SideA with 2 circuits ERC checked
Parts:
- added C?: CP1, symbol CP1
- added D? (x3): LED, symbol LED
- added Q? (x3): BC237, TO92-EBC, symbol BC237
- added R? (x6): R, symbol R
- added SW? (x3): SW_PUSH, symbol SW_PUSH
Connections:
- net labels added: +5V, GND
- wire segments 0 -> 40
Other:
- note added: "Memory\n"
- note added: "Time delay switch"
