File: sideB.sch (KiCad schematic (older format))
At the start: 39 parts, among them IC1 4520, IC2 LM2902N, IC3 LM555N, J1 USB_2, P1 CONN_2, Q4 NPN, SW4 SW_PUSH

Commit message: Edited transistor pinout. Created new compoment NPN.
Changed lines of the file:
@@
-EESchema Schematic File Version 2  date Thu 14 Feb 2013 10:34:18 CET
+EESchema Schematic File Version 2  date Tue 26 Feb 2013 22:34:39 CET
 LIBS:power
 LIBS:device
@@
 LIBS:contrib
 LIBS:valves
+LIBS:npn
 LIBS:sideB-cache
 EELAYER 25  0
@@
 Sheet 1 1
 Title "SMT4dummies - sideB"
-Date "14 feb 2013"
+Date "26 feb 2013"
 Rev "1"
 Comp "d-Squared Robotics"
@@
 Comment4 ""
 $EndDescr
+$Comp
+L NPN Q4
+U 1 1 512D2A5C
+P 5500 5000
+F 0 "Q4" H 5500 4850 50  0000 R CNN
+F 1 "NPN" H 5500 5150 50  0000 R CNN
+	1    5500 5000
+	1    0    0    -1
+$EndComp
 Wire Wire Line
 	2700 5400 2700 5250
@@
 	2700 5250 2950 5250
 Wire Wire Line
-	5050 5950 5050 5850
+	5050 5850 5050 5950
 Wire Wire Line
 	3650 5700 3650 5600
@@
 	800  2500 800  1600
 Wire Wire Line
-	1450 2150 1450 2050
-Wire Wire Line
-	1250 2150 1450 2150
+	1450 2050 1450 2150
+Wire Wire Line
+	1450 2150 1250 2150
 Connection ~ 1350 2150
 Wire Wire Line
@@
 	6600 2650 6600 2500
 Wire Wire Line
-	7800 1050 8350 1050
+	8350 1050 7800 1050
 Connection ~ 7800 2050
 Wire Wire Line
@@
 	1    0    0    -1
 $EndComp
-$Comp
-L NPN Q4
-U 1 1 5053179A
-P 5500 5000
-F 0 "Q4" H 5500 4850 50  0000 R CNN
-F 1 "NPN" H 5500 5150 50  0000 R CNN
-	1    5500 5000
-	1    0    0    -1
-$EndComp

Commit message: LED resistors value (150ohm) added to schematics.
Parts:
- R10, R11, R12, R13, R19, R20, R21, R22, R23: value R -> 150R
Changed lines of the file:
@@
-EESchema Schematic File Version 2  date Tue 26 Feb 2013 22:34:39 CET
+EESchema Schematic File Version 2  date Tue 26 Feb 2013 22:59:04 CET
 LIBS:power
 LIBS:device
@@
 P 5600 4500
 F 0 "R23" V 5680 4500 50  0000 C CNN
-F 1 "R" V 5600 4500 50  0000 C CNN
+F 1 "150R" V 5600 4500 50  0000 C CNN
 	1    5600 4500
 	1    0    0    -1
@@
 P 10200 2700
 F 0 "R21" V 10280 2700 50  0000 C CNN
-F 1 "R" V 10200 2700 50  0000 C CNN
+F 1 "150R" V 10200 2700 50  0000 C CNN
 	1    10200 2700
 	0    1    1    0
@@
 P 10200 3250
 F 0 "R22" V 10280 3250 50  0000 C CNN
-F 1 "R" V 10200 3250 50  0000 C CNN
+F 1 "150R" V 10200 3250 50  0000 C CNN
 	1    10200 3250
 	0    1    1    0
@@
 P 10200 2150
 F 0 "R20" V 10280 2150 50  0000 C CNN
-F 1 "R" V 10200 2150 50  0000 C CNN
+F 1 "150R" V 10200 2150 50  0000 C CNN
 	1    10200 2150
 	0    1    1    0
@@
 P 10200 1550
 F 0 "R19" V 10280 1550 50  0000 C CNN
-F 1 "R" V 10200 1550 50  0000 C CNN
+F 1 "150R" V 10200 1550 50  0000 C CNN
 	1    10200 1550
 	0    1    1    0
@@
 P 5300 2300
 F 0 "R12" V 5380 2300 50  0000 C CNN
-F 1 "R" V 5300 2300 50  0000 C CNN
+F 1 "150R" V 5300 2300 50  0000 C CNN
 	1    5300 2300
 	1    0    0    -1
@@
 P 5600 2300
 F 0 "R13" V 5680 2300 50  0000 C CNN
-F 1 "R" V 5600 2300 50  0000 C CNN
+F 1 "150R" V 5600 2300 50  0000 C CNN
 	1    5600 2300
 	1    0    0    -1
@@
 P 5050 2300
 F 0 "R11" V 5130 2300 50  0000 C CNN
-F 1 "R" V 5050 2300 50  0000 C CNN
+F 1 "150R" V 5050 2300 50  0000 C CNN
 	1    5050 2300
 	1    0    0    -1
@@
 P 4750 2300
 F 0 "R10" V 4830 2300 50  0000 C CNN
-F 1 "R" V 4750 2300 50  0000 C CNN
+F 1 "150R" V 4750 2300 50  0000 C CNN
 	1    4750 2300
 	1    0    0    -1

Commit message: Added values for resistors.
Parts:
- R14, R15, R16, R17, R18: value R -> 1K
- RV1: value POT -> 100K
Changed lines of the file:
@@
-EESchema Schematic File Version 2  date Tue 26 Feb 2013 22:59:04 CET
+EESchema Schematic File Version 2  date Wed 27 Feb 2013 15:26:14 CET
 LIBS:power
 LIBS:device
@@
 Sheet 1 1
 Title "SMT4dummies - sideB"
-Date "26 feb 2013"
+Date "27 feb 2013"
 Rev "1"
 Comp "d-Squared Robotics"
@@
 Wire Notes Line
 	6050 750  6050 3200
-Connection ~ 3100 1700
 Connection ~ 2550 1700
 Wire Wire Line
@@
 P 6600 2250
 F 0 "RV1" H 6600 2150 50  0000 C CNN
-F 1 "POT" H 6600 2250 50  0000 C CNN
+F 1 "100K" H 6600 2250 50  0000 C CNN
 	1    6600 2250
 	0    1    1    0
@@
 P 7550 1300
 F 0 "R14" V 7630 1300 50  0000 C CNN
-F 1 "R" V 7550 1300 50  0000 C CNN
+F 1 "1K" V 7550 1300 50  0000 C CNN
 	1    7550 1300
 	1    0    0    -1
@@
 P 7550 3100
 F 0 "R17" V 7630 3100 50  0000 C CNN
-F 1 "R" V 7550 3100 50  0000 C CNN
+F 1 "1K" V 7550 3100 50  0000 C CNN
 	1    7550 3100
 	1    0    0    -1
@@
 P 7550 3700
 F 0 "R18" V 7630 3700 50  0000 C CNN
-F 1 "R" V 7550 3700 50  0000 C CNN
+F 1 "1K" V 7550 3700 50  0000 C CNN
 	1    7550 3700
 	1    0    0    -1
@@
 P 7550 2500
 F 0 "R16" V 7630 2500 50  0000 C CNN
-F 1 "R" V 7550 2500 50  0000 C CNN
+F 1 "1K" V 7550 2500 50  0000 C CNN
 	1    7550 2500
 	1    0    0    -1
@@
 P 7550 1900
 F 0 "R15" V 7630 1900 50  0000 C CNN
-F 1 "R" V 7550 1900 50  0000 C CNN
+F 1 "1K" V 7550 1900 50  0000 C CNN
 	1    7550 1900
 	1    0    0    -1

Commit message: All components spitted on the board.
Parts:
- added unit 2 of IC1
Connections:
- net +5V: now also IC1.16 (VDD)
- net GND: now also IC1.8 (VSS), IC1.9 (CK)
- no-connect marks 2 -> 6
Other:
- moved on the sheet: D4, D5, D6, D7, R10, R11, R12, R13, R9, SW4

Commit message: Modified counter.
Connections:
- net GND: now also IC1.10 (Enable), IC1.15 (Reset)
