File: SMT4dummies.sch (KiCad schematic (older format))
At the start: 0 parts

Commit message: Merged both sides
Parts:
- added C1: CP1, symbol CP1
- added C2: 0.1uF, symbol C
- added D1, D10, D11, D12, D2, D3, D4, D5, D6, D7, D8, D9: LED, symbol LED
- added D13, D14: 1N4148, symbol DIODE
- added IC1: 4520, symbol 4520
- added IC2: LM2902N, symbol LM2902N
- added IC3: LM555N, symbol LM555N
- added J1: USB_2, symbol USB_2
- added P1: CONN_2, symbol CONN_2
- added Q1, Q2, Q3, Q4: NPN, symbol NPN
- added R1, R10, R11, R12, R13, R14, R15, R16, R17, R18, R19, R2, R20, R21, R22, R23, R3, R4, R5, R6: R, symbol R
- added R24, R25: 1K, symbol R
- added R8, R9: 4.7K, symbol R
- added RV1: POT, symbol POT
- added RV2: 100K, symbol POT
- added SW1, SW2, SW3, SW4: SW_PUSH, symbol SW_PUSH
Connections:
- new net: D7.1 (A), IC1.3 (Q1)
- new net: D6.1 (A), IC1.4 (Q2)
- new net: D5.1 (A), IC1.5 (Q3)
- new net: D4.1 (A), IC1.6 (Q4)
- new net: D4.2 (K), R10.1
- new net: D5.2 (K), R11.1
- new net: D7.2 (K), R13.1
- new net: D6.2 (K), R12.1
- new net: D8.1 (A), IC2.1
- new net: IC2.2 (-), R14.2, R15.1
- new net: IC2.6 (-), R15.2, R16.1
- new net: D9.1 (A), IC2.7
- new net: D10.1 (A), IC2.8
- new net: IC2.9 (-), R16.2, R17.1
- new net: IC2.13 (-), R17.2, R18.1
- new net: D11.1 (A), IC2.14
- new net: D8.2 (K), R19.2
- new net: D9.2 (K), R20.2
- new net: D11.2 (K), R22.2
- new net: D10.2 (K), R21.2
- new net: IC3.3 (Q), R25.2
- new net: D13.2 (K), RV2.1
- new net: D14.1 (A), RV2.3
- new net: Q4.2 (B), R25.1
- new net: Q4.3 (C), R23.2
- new net: D12.2 (K), R23.1
- new net: Q3.2 (B), R5.1, SW3.2
- new net: Q3.3 (C), R4.1, R6.2
- new net: Q2.2 (B), R4.2, SW2.2
- new net: Q2.3 (C), R3.2, R5.2
- new net: Q1.2 (B), R1.1
- new net: Q1.3 (C), R2.2
- new net: D3.2 (K), R6.1
- new net: D2.2 (K), R3.1
- new net: C1.1, R1.2, SW1.1
- new net: D1.2 (K), R2.1
- new net +5V: D1.1 (A), D12.1 (A), D2.1 (A), D3.1 (A), IC1.16 (VDD), IC1.2 (Enable), IC2.4 (V+), IC3.4 (R), IC3.8 (VCC), J1.1, P1.1 (P1), R14.1, R24.2, R8.2, RV1.1, SW1.2, SW4.1
- new net ANLG_INPUT: IC2.10 (+), IC2.12 (+), IC2.3 (+), IC2.5 (+), RV1.2
- new net CLK: IC1.1 (CK), R9.1, SW4.2
- new net DIS: IC3.7 (DIS), R24.1, RV2.2
- new net GND: C1.2, C2.2, IC1.7 (Reset), IC1.8 (VSS), IC2.11 (V-), IC3.1 (GND), IC3.5 (CV), J1.4, P1.2 (PM), Q1.1 (E), Q2.1 (E), Q3.1 (E), Q4.1 (E), R10.2, R11.2, R12.2, R13.2, R18.2, R19.1, R20.1, R21.1, R22.1, R8.1, R9.2, RV1.3, SW2.1, SW3.1
- new net THR: C2.1, D13.1 (A), D14.2 (K), IC3.2 (TR), IC3.6 (THR)
- no-connect marks 0 -> 2
Other:
- note added: "4 bits ADC"
- note added: "555-based PWM dimmer"
- note added: "KiCad needs this"
- note added: "Memory\n"
- note added: "Power supply"
- note added: "Push-switch operated 4-bit up binary counter"
- note added: "Time delay switch"

Commit message: Modified counter.
Parts:
- added unit 2 of IC1
- R10, R11, R12, R13: value R -> 150R
Connections:
- net +5V: now also IC1.16 (VDD)
- net GND: now also IC1.10 (Enable), IC1.15 (Reset), IC1.8 (VSS), IC1.9 (CK)
- no-connect marks 2 -> 6

Commit message: Track problems solved.
Parts:
- removed R8: 4.7K, symbol R
Changed lines of the file:
@@
-EESchema Schematic File Version 2  date Mon 04 Mar 2013 13:15:41 CET
+EESchema Schematic File Version 2  date Mon 04 Mar 2013 14:08:08 CET
 LIBS:power
 LIBS:device
@@
 Comment4 ""
 $EndDescr
+Wire Wire Line
+	2600 1650 2600 1700
 Connection ~ 2350 2800
 Wire Wire Line
-	2350 2950 2350 2600
+	2350 2600 2350 2950
 Wire Wire Line
 	5300 5000 5100 5000
@@
 Connection ~ 2400 5200
 Wire Wire Line
-	2400 5300 2400 5000
+	2400 5000 2400 5300
 Wire Wire Line
 	2400 5700 2400 5800
@@
 	7550 3950 7550 4050
 Wire Wire Line
-	7550 2850 7550 2750
+	7550 2750 7550 2850
 Wire Wire Line
 	7550 1550 7550 1650
@@
 	10850 4150 6250 4150
 Wire Wire Line
-	1900 5000 2950 5000
+	2950 5000 1900 5000
 Connection ~ 2700 5000
 Wire Wire Line
@@
 	1700 750  800  750
 Wire Wire Line
-	1250 1850 1450 1850
+	1450 1850 1250 1850
 Wire Wire Line
 	1350 2250 1350 2150
@@
 	7700 5800 7800 5800
 Wire Wire Line
-	7100 5500 7100 5900
+	7100 5900 7100 5500
 Wire Wire Line
 	6500 5200 6600 5200
@@
 	6600 5400 6450 5400
 Wire Wire Line
-	9250 5350 9250 5800
+	9250 5800 9250 5350
 Wire Wire Line
 	9250 4750 9250 4850
@@
 	10200 5500 10750 5500
 Wire Wire Line
-	10750 5350 10750 5800
+	10750 5800 10750 5350
 Connection ~ 10750 5500
 Wire Wire Line
@@
 	10750 6850 10750 6200
 Wire Wire Line
-	9600 6750 9600 6850
+	9600 6850 9600 6750
 Connection ~ 9600 6850
 Wire Wire Line
@@
 	3500 1200 3500 1100
 Wire Wire Line
-	2500 1700 3050 1700
-Wire Wire Line
-	3050 1700 3050 1650
-Wire Wire Line
-	2500 1750 2500 1600
+	3050 1650 3050 1700
 Wire Wire Line
 	2800 1600 2800 1550
@@
 Wire Wire Line
 	2800 1550 3050 1550
-Wire Wire Line
-	2500 2300 2500 2250
-Connection ~ 2500 1700
 Wire Notes Line
 	6000 750  6000 3200
@@
 	5200 1450 4250 1450
 Connection ~ 2350 2700
+Wire Wire Line
+	3050 1700 2600 1700
 $Comp
 L 4520 IC1
@@
 L +5V #PWR08
 U 1 1 51348E9A
-P 2500 1600
-F 0 "#PWR08" H 2500 1690 20  0001 C CNN
-F 1 "+5V" H 2500 1690 30  0000 C CNN
-	1    2500 1600
-	1    0    0    -1
-$EndComp
-$Comp
-L R R8
-U 1 1 51348E99
-P 2500 2000
-F 0 "R8" V 2580 2000 50  0000 C CNN
-F 1 "4.7K" V 2500 2000 50  0000 C CNN
-	1    2500 2000
-	-1   0    0    1
-$EndComp
-$Comp
-L GND #PWR09
-U 1 1 51348E98
-P 2500 2300
-F 0 "#PWR09" H 2500 2300 30  0001 C CNN
-F 1 "GND" H 2500 2230 30  0001 C CNN
-	1    2500 2300
+P 2600 1650
+F 0 "#PWR08" H 2600 1740 20  0001 C CNN
+F 1 "+5V" H 2600 1740 30  0000 C CNN
+	1    2600 1650
 	1    0    0    -1
 $EndComp
@@
 Push-switch operated 4-bit up binary counter
 $Comp
-L +5V #PWR010
+L +5V #PWR09
 U 1 1 51348E97
 P 3500 1100
-F 0 "#PWR010" H 3500 1190 20  0001 C CNN
+F 0 "#PWR09" H 3500 1190 20  0001 C CNN
 F 1 "+5V" H 3500 1190 30  0000 C CNN
 	1    3500 1100
@@
 $EndComp
 $Comp
-L GND #PWR011
+L GND #PWR010
 U 1 1 51348E96
 P 3500 1950
-F 0 "#PWR011" H 3500 1950 30  0001 C CNN
+F 0 "#PWR010" H 3500 1950 30  0001 C CNN
 F 1 "GND" H 3500 1880 30  0001 C CNN
 	1    3500 1950
@@
 $EndComp
 $Comp
-L GND #PWR012
+L GND #PWR011
 U 1 1 51348E94
 P 2350 2950
-F 0 "#PWR012" H 2350 2950 30  0001 C CNN
+F 0 "#PWR011" H 2350 2950 30  0001 C CNN
 F 1 "GND" H 2350 2880 30  0001 C CNN
 	1    2350 2950
@@
 $EndComp
 $Comp
-L +5V #PWR013
+L +5V #PWR012
 U 1 1 512B78F9
 P 6500 5200
-F 0 "#PWR013" H 6500 5290 20  0001 C CNN
+F 0 "#PWR012" H 6500 5290 20  0001 C CNN
 F 1 "+5V" H 6500 5290 30  0000 C CNN
 	1    6500 5200
@@
 $EndComp
 $Comp
-L GND #PWR014
+L GND #PWR013
 U 1 1 512B78F8
 P 6450 5400
-F 0 "#PWR014" H 6450 5400 30  0001 C CNN
+F 0 "#PWR013" H 6450 5400 30  0001 C CNN
 F 1 "GND" H 6450 5330 30  0001 C CNN
 	1    6450 5400
@@
 $EndComp
 $Comp
-L +5V #PWR015
+L +5V #PWR014
 U 1 1 512B78F3
 P 8650 5300
-F 0 "#PWR015" H 8650 5390 20  0001 C CNN
+F 0 "#PWR014" H 8650 5390 20  0001 C CNN
 F 1 "+5V" H 8650 5390 30  0000 C CNN
 	1    8650 5300
@@
 $EndComp
 $Comp
-L GND #PWR016
+L GND #PWR015
 U 1 1 512B78F2
 P 8600 5500
-F 0 "#PWR016" H 8600 5500 30  0001 C CNN
+F 0 "#PWR015" H 8600 5500 30  0001 C CNN
 F 1 "GND" H 8600 5430 30  0001 C CNN
 	1    8600 5500
@@
 $EndComp
 $Comp
-L +5V #PWR017
+L +5V #PWR016
 U 1 1 511BD2C7
 P 4200 5900
-F 0 "#PWR017" H 4200 5990 20  0001 C CNN
+F 0 "#PWR016" H 4200 5990 20  0001 C CNN
 F 1 "+5V" H 4200 5990 30  0000 C CNN
 	1    4200 5900
@@
 DIS
 $Comp
-L GND #PWR018
+L GND #PWR017
 U 1 1 5059F5FF
 P 3650 5700
-F 0 "#PWR018" H 3650 5700 30  0001 C CNN
+F 0 "#PWR017" H 3650 5700 30  0001 C CNN
 F 1 "GND" H 3650 5630 30  0001 C CNN
 	1    3650 5700
@@
 $EndComp
 $Comp
-L +5V #PWR019
+L +5V #PWR018
 U 1 1 5059F5F6
 P 3650 4700
-F 0 "#PWR019" H 3650 4790 20  0001 C CNN
+F 0 "#PWR018" H 3650 4790 20  0001 C CNN
 F 1 "+5V" H 3650 4790 30  0000 C CNN
 	1    3650 4700
@@
 $EndComp
 $Comp
-L +5V #PWR020
+L +5V #PWR019
 U 1 1 5059D843
 P 6850 2900
-F 0 "#PWR020" H 6850 2990 20  0001 C CNN
+F 0 "#PWR019" H 6850 2990 20  0001 C CNN
 F 1 "+5V" H 6850 2990 30  0000 C CNN
 	1    6850 2900
@@
 $EndComp
 $Comp
-L GND #PWR021
+L GND #PWR020
 U 1 1 5059D836
 P 6850 3900
-F 0 "#PWR021" H 6850 3900 30  0001 C CNN
+F 0 "#PWR020" H 6850 3900 30  0001 C CNN
 F 1 "GND" H 6850 3830 30  0001 C CNN
 	1    6850 3900
@@
 $EndComp
 $Comp
-L GND #PWR022
+L GND #PWR021
 U 1 1 505317F2
 P 5600 5750
-F 0 "#PWR022" H 5600 5750 30  0001 C CNN
+F 0 "#PWR021" H 5600 5750 30  0001 C CNN
 F 1 "GND" H 5600 5680 30  0001 C CNN
 	1    5600 5750
@@
 $EndComp
 $Comp
-L +5V #PWR023
+L +5V #PWR022
 U 1 1 505317DA
 P 5600 3750
-F 0 "#PWR023" H 5600 3840 20  0001 C CNN
+F 0 "#PWR022" H 5600 3840 20  0001 C CNN
 F 1 "+5V" H 5600 3840 30  0000 C CNN
 	1    5600 3750
@@
 Power supply
 $Comp
-L +5V #PWR024
+L +5V #PWR023
 U 1 1 5052243B
 P 1350 1750
-F 0 "#PWR024" H 1350 1840 20  0001 C CNN
+F 0 "#PWR023" H 1350 1840 20  0001 C CNN
 F 1 "+5V" H 1350 1840 30  0000 C CNN
 	1    1350 1750
@@
 $EndComp
 $Comp
-L GND #PWR025
+L GND #PWR024
 U 1 1 5052242C
 P 1350 2250
-F 0 "#PWR025" H 1350 2250 30  0001 C CNN
+F 0 "#PWR024" H 1350 2250 30  0001 C CNN
 F 1 "GND" H 1350 2180 30  0001 C CNN
 	1    1350 2250
@@
 $EndComp
 $Comp
-L GND #PWR026
+L GND #PWR025
 U 1 1 50521A79
 P 2400 5800
-F 0 "#PWR026" H 2400 5800 30  0001 C CNN
+F 0 "#PWR025" H 2400 5800 30  0001 C CNN
 F 1 "GND" H 2400 5730 30  0001 C CNN
 	1    2400 5800
@@
 KiCad needs this
 $Comp
-L PWR_FLAG #FLG027
+L PWR_FLAG #FLG026
 U 1 1 505219BA
 P 1000 1050
-F 0 "#FLG027" H 1000 1320 30  0001 C CNN
+F 0 "#FLG026" H 1000 1320 30  0001 C CNN
 F 1 "PWR_FLAG" H 1000 1280 30  0000 C CNN
 	1    1000 1050
@@
 $EndComp
 $Comp
-L PWR_FLAG #FLG028
+L PWR_FLAG #FLG027
 U 1 1 505219B5
 P 1350 1100
-F 0 "#FLG028" H 1350 1370 30  0001 C CNN
+F 0 "#FLG027" H 1350 1370 30  0001 C CNN
 F 1 "PWR_FLAG" H 1350 1330 30  0000 C CNN
 	1    1350 1100
@@
 $EndComp
 $Comp
-L GND #PWR029
+L GND #PWR028
 U 1 1 5052199C
 P 1350 1200
-F 0 "#PWR029" H 1350 1200 30  0001 C CNN
+F 0 "#PWR028" H 1350 1200 30  0001 C CNN
 F 1 "GND" H 1350 1130 30  0001 C CNN
 	1    1350 1200
@@
 $EndComp
 $Comp
-L +5V #PWR030
+L +5V #PWR029
 U 1 1 50521991
 P 1000 950
-F 0 "#PWR030" H 1000 1040 20  0001 C CNN
+F 0 "#PWR029" H 1000 1040 20  0001 C CNN
 F 1 "+5V" H 1000 1040 30  0000 C CNN
 	1    1000 950
@@
 THR
 $Comp
-L GND #PWR031
+L GND #PWR030
 U 1 1 505217B9
 P 2700 5400
-F 0 "#PWR031" H 2700 5400 30  0001 C CNN
+F 0 "#PWR030" H 2700 5400 30  0001 C CNN
 F 1 "GND" H 2700 5330 30  0001 C CNN
 	1    2700 5400
@@
 4 bits ADC
 $Comp
-L GND #PWR032
+L GND #PWR031
 U 1 1 5051AA37
 P 6600 2650
-F 0 "#PWR032" H 6600 2650 30  0001 C CNN
+F 0 "#PWR031" H 6600 2650 30  0001 C CNN
 F 1 "GND" H 6600 2580 30  0001 C CNN
 	1    6600 2650
@@
 $EndComp
 $Comp
-L +5V #PWR033
+L +5V #PWR032
 U 1 1 5051AA2B
 P 6600 1900
-F 0 "#PWR033" H 6600 1990 20  0001 C CNN
+F 0 "#PWR032" H 6600 1990 20  0001 C CNN
 F 1 "+5V" H 6600 1990 30  0000 C CNN
 	1    6600 1900
@@
 ANLG_INPUT
 $Comp
-L +5V #PWR034
+L +5V #PWR033
 U 1 1 5051A869
 P 7550 950
-F 0 "#PWR034" H 7550 1040 20  0001 C CNN
+F 0 "#PWR033" H 7550 1040 20  0001 C CNN
 F 1 "+5V" H 7550 1040 30  0000 C CNN
 	1    7550 950
@@
 $EndComp
 $Comp
-L GND #PWR035
+L GND #PWR034
 U 1 1 5051A85F
 P 7550 4050
-F 0 "#PWR035" H 7550 4050 30  0001 C CNN
+F 0 "#PWR034" H 7550 4050 30  0001 C CNN
 F 1 "GND" H 7550 3980 30  0001 C CNN
 	1    7550 4050
@@
 $EndComp
 $Comp
-L GND #PWR036
+L GND #PWR035
 U 1 1 5051A7F3
 P 10600 2750
-F 0 "#PWR036" H 10600 2750 30  0001 C CNN
+F 0 "#PWR035" H 10600 2750 30  0001 C CNN
 F 1 "GND" H 10600 2680 30  0001 C CNN
 	1    10600 2750
@@
 $EndComp
 $Comp
-L GND #PWR037
+L GND #PWR036
 U 1 1 5051A7F2
 P 10600 3300
-F 0 "#PWR037" H 10600 3300 30  0001 C CNN
+F 0 "#PWR036" H 10600 3300 30  0001 C CNN
 F 1 "GND" H 10600 3230 30  0001 C CNN
 	1    10600 3300
@@
 $EndComp
 $Comp
-L GND #PWR038
+L GND #PWR037
 U 1 1 5051A7C6
 P 10600 2200
-F 0 "#PWR038" H 10600 2200 30  0001 C CNN
+F 0 "#PWR037" H 10600 2200 30  0001 C CNN
 F 1 "GND" H 10600 2130 30  0001 C CNN
 	1    10600 2200
@@
 $EndComp
 $Comp
-L GND #PWR039
+L GND #PWR038
 U 1 1 5051A766
 P 10600 1600
-F 0 "#PWR039" H 10600 1600 30  0001 C CNN
+F 0 "#PWR038" H 10600 1600 30  0001 C CNN
 F 1 "GND" H 10600 1530 30  0001 C CNN
 	1    10600 1600
